File: vssop_10_breakout.sch (KiCad schematic (older format))
At the start: 3 parts, among them J1 CONN_01X05, J2 CONN_01X05, U1 VSSOP-10

Commit message: Replace VSSOP footprint with custom one
Parts:
- U1: footprint Housings_SSOP:TSSOP-10_3x3mm_Pitch0.5mm -> VSSOP:VSSOP-10_3x3mm_Pitch0.5mm
Changed lines of the file:
@@
 LIBS:valves
 LIBS:vssop-10
+LIBS:vssop_10_breakout-cache
 EELAYER 25 0
 EELAYER END
@@
 F 0 "U1" H 5950 3100 60  0000 C CNN
 F 1 "VSSOP-10" H 5950 3800 60  0000 C CNN
-F 2 "Housings_SSOP:TSSOP-10_3x3mm_Pitch0.5mm" H 5950 3800 60  0001 C CNN
+F 2 "VSSOP:VSSOP-10_3x3mm_Pitch0.5mm" H 5950 3800 60  0001 C CNN
 F 3 "" H 5950 3800 60  0001 C CNN
 	1    5950 3800
